Commit message: minor changes

File: tp-final/adaptive_gripper/mycobot_adaptive_gripper.urdf (robot description, URDF)
Before this commit: robot adaptive_gripper, 7 links, 6 joints
Links:
- link gripper_base: mass None -> 0.03
- link gripper_left1: mass None -> 0.008
- link gripper_left2: mass None -> 0.008
- link gripper_left3: mass None -> 0.008
- link gripper_right1: mass None -> 0.008
- link gripper_right2: mass None -> 0.008
- link gripper_right3: mass None -> 0.008

File: tp-final/mycobot_320_m5_2022.xacro (robot description, xacro)
@@ -14,4 +14,6 @@
   <xacro:property name="link6_mass" value="0.0739" />
   <xacro:property name="flange_mass" value="0.035" />
+  <xacro:property name="gripper_base_mass" value="0.03" />
+  <xacro:property name="gripper_finger_mass" value="0.008" />
   <xacro:macro name="link_inertial" params="xg yg zg mass ixx iyy izz">
     <inertial>
@@ -190,4 +192,6 @@
   </joint>
   <link name="gripper_base">
+    <xacro:link_inertial xg="0" yg="0" zg="-0.012" mass="${gripper_base_mass}" ixx="0.00001"
+      iyy="0.00001" izz="0.00001" />
     <visual>
       <geometry>
@@ -204,4 +208,6 @@
   </link>
   <link name="gripper_left1">
+    <xacro:link_inertial xg="0.039" yg="-0.0133" zg="-0.012" mass="${gripper_finger_mass}"
+      ixx="0.000002" iyy="0.000002" izz="0.000002" />
     <visual>
       <geometry>
@@ -218,4 +224,6 @@
   </link>
   <link name="gripper_left2">
+    <xacro:link_inertial xg="0.005" yg="-0.0195" zg="-0.012" mass="${gripper_finger_mass}"
+      ixx="0.000002" iyy="0.000002" izz="0.000002" />
     <visual>
       <geometry>
@@ -232,4 +240,6 @@
   </link>
   <link name="gripper_left3">
+    <xacro:link_inertial xg="0.012" yg="0.0025" zg="-0.012" mass="${gripper_finger_mass}"
+      ixx="0.000002" iyy="0.000002" izz="0.000002" />
     <visual>
       <geometry>
@@ -246,4 +256,6 @@
   </link>
   <link name="gripper_right1">
+    <xacro:link_inertial xg="-0.039" yg="-0.0133" zg="-0.012" mass="${gripper_finger_mass}"
+      ixx="0.000002" iyy="0.000002" izz="0.000002" />
     <visual>
       <geometry>
@@ -260,4 +272,6 @@
   </link>
   <link name="gripper_right2">
+    <xacro:link_inertial xg="-0.005" yg="-0.0195" zg="-0.012" mass="${gripper_finger_mass}"
+      ixx="0.000002" iyy="0.000002" izz="0.000002" />
     <visual>
       <geometry>
@@ -274,4 +288,6 @@
   </link>
   <link name="gripper_right3">
+    <xacro:link_inertial xg="-0.012" yg="0.0025" zg="-0.012" mass="${gripper_finger_mass}"
+      ixx="0.000002" iyy="0.000002" izz="0.000002" />
     <visual>
       <geometry>

Commit message: fix paths

File: tp-final/adaptive_gripper/mycobot_adaptive_gripper.urdf (robot description, URDF)
Before this commit: robot adaptive_gripper, 7 links, 6 joints
Links:
- link gripper_base: geometry collision mesh filename=package://clase5/robot_description/adaptive_gripper/gripper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; visual mesh filename=package://clase5/robot_description/adaptive_gripper/gripper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
- link gripper_left1: geometry collision mesh filename=package://clase5/robot_description/adaptive_gripper/gripper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; visual mesh filename=package://clase5/robot_description/adaptive_gripper/gripper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
- link gripper_left2: geometry collision mesh filename=package://clase5/robot_description/adaptive_gripper/gripper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; visual mesh filename=package://clase5/robot_description/adaptive_gripper/gripper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
- link gripper_left3: geometry collision mesh filename=package://clase5/robot_description/adaptive_gripper/gripper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; visual mesh filename=package://clase5/robot_description/adaptive_gripper/gripper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
- link gripper_right1: geometry collision mesh filename=package://clase5/robot_description/adaptive_gripper/gripper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; visual mesh filename=package://clase5/robot_description/adaptive_gripper/gripper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
- link gripper_right2: geometry collision mesh filename=package://clase5/robot_description/adaptive_gripper/gripper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; visual mesh filename=package://clase5/robot_description/adaptive_gripper/gripper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
- link gripper_right3: geometry collision mesh filename=package://clase5/robot_description/adaptive_gripper/gripper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; visual mesh filename=package://clase5/robot_description/adaptive_gripper/gripper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
