Commit message: minor changes

File: tp-final/clase5/robot_description/mycobot_320_m5_2022/mycobot_320_m5_2022.xacro (robot description, xacro)
@@ -355,4 +355,53 @@
     <mimic joint="gripper_controller" multiplier="1.0" offset="0" />
   </joint>
+  <!--  TCP / PUNTO DE AGARRE *******************-->
+  <!-- El eje de aproximacion de la pinza es el +y de link6: con todas las
+       juntas en cero el brazo apunta hacia arriba y ese +y queda mirando
+       hacia abajo. La pinza ocupa y de -0.029 a +0.042 en ese frame, asi que
+       tool0 se coloca 13mm mas alla de la punta.
+       La rotacion -90 en x hace que el +z de tool0 sea el eje de
+       aproximacion, que es la convencion que espera MoveIt. -->
+  <xacro:property name="tool0_offset" value="0.055" />
+  <link name="tool0" />
+  <joint name="link6_to_tool0" type="fixed">
+    <parent link="link6" />
+    <child link="tool0" />
+    <origin xyz="0 ${tool0_offset} 0" rpy="-1.5708 0 0" />
+  </joint>
+  <!--  ROS2 CONTROL *******************-->
+  <!-- Sin este bloque no existe el controller_manager, y entonces los
+       spawners de mycobot_launch.py (joint_state_broadcaster y
+       joint_trajectory_controller) no tienen contra que levantar: MoveIt
+       puede planificar pero no ejecutar. Las interfaces son de esfuerzo
+       porque ros2_controllers.yaml ya define las ganancias PID por junta. -->
+  <xacro:arg name="controllers_file" default="$(find clase5)/config/mycobot_320_m5_2022/ros2_controllers.yaml" />
+  <xacro:macro name="joint_control" params="joint">
+    <joint name="${joint}">
+      <command_interface name="effort">
+        <param name="min">-${joint_effort}</param>
+        <param name="max">${joint_effort}</param>
+      </command_interface>
+      <state_interface name="position" />
+      <state_interface name="velocity" />
+      <state_interface name="effort" />
+    </joint>
+  </xacro:macro>
+  <ros2_control name="GazeboSimSystem" type="system">
+    <hardware>
+      <plugin>gz_ros2_control/GazeboSimSystem</plugin>
+    </hardware>
+    <xacro:joint_control joint="joint1" />
+    <xacro:joint_control joint="joint2" />
+    <xacro:joint_control joint="joint3" />
+    <xacro:joint_control joint="joint4" />
+    <xacro:joint_control joint="joint5" />
+    <xacro:joint_control joint="joint6" />
+  </ros2_control>
+  <gazebo>
+    <plugin filename="gz_ros2_control-system"
+      name="gz_ros2_control::GazeboSimROS2ControlPlugin">
+      <parameters>$(arg controllers_file)</parameters>
+    </plugin>
+  </gazebo>
   <!-- CONFIGURACION DE PLUGINS DE GAZEBO  *******************-->
   <xacro:macro name="apply_joint_force" params="joint">

Commit message: more minor changes

File: tp-final/clase5/robot_description/mycobot_320_m5_2022/mycobot_320_m5_2022.xacro (robot description, xacro)
@@ -4,6 +4,6 @@
   <xacro:property name="joint_effort" value="56.0" />
   <xacro:property name="joint_velocity" value="2.792527" />
-  <xacro:property name="joint_damping" value="0.0" />
-  <xacro:property name="joint_friction" value="0.0" />
+  <xacro:property name="joint_damping" value="1.0" />
+  <xacro:property name="joint_friction" value="0.5" />
   <xacro:property name="base_mass" value="0.12" />
   <xacro:property name="link1_mass" value="0.12" />
@@ -42,7 +42,7 @@
     <collision>
       <geometry>
-        <mesh filename="package://clase5/robot_description/mycobot_320_m5_2022/base.dae" />
-      </geometry>
-      <origin xyz="0.0 0 0 " rpy=" 0 0 1.5708" />
+        <box size="0.11712 0.14372 0.1104" />
+      </geometry>
+      <origin xyz="-0.01064 0.00002 0.05538" rpy="0 0 1.5708" />
     </collision>
   </link>
@@ -58,7 +58,7 @@
     <collision>
       <geometry>
-        <mesh filename="package://clase5/robot_description/mycobot_320_m5_2022/link1.dae" />
-      </geometry>
-      <origin xyz="0.0 0.0 -0.078 " rpy=" 0 0 1.5708" />
+        <box size="0.1114 0.07697 0.11769" />
+      </geometry>
+      <origin xyz="-0.00005 -0.01817 -0.01896" rpy="0 0 1.5708" />
     </collision>
   </link>
@@ -74,7 +74,7 @@
     <collision>
       <geometry>
-        <mesh filename="package://clase5/robot_description/mycobot_320_m5_2022/link2.dae" />
-      </geometry>
-      <origin xyz="0.0 0.0 -0.04 " rpy=" 0 1.5708 0" />
+        <box size="0.09742 0.07633 0.20834" />
+      </geometry>
+      <origin xyz="0.06589 0.00031 -0.01632" rpy="0 1.5708 0" />
     </collision>
   </link>
@@ -90,7 +90,7 @@
     <collision>
       <geometry>
-        <mesh filename="package://clase5/robot_description/mycobot_320_m5_2022/link3.dae" />
-      </geometry>
-      <origin xyz="0.0 0.0 0.039 " rpy=" 1.5708 1.5708 1.5708" />
+        <box size="0.087 0.06903 0.18483" />
+      </geometry>
+      <origin xyz="0.05779 0.00028 0.00755" rpy="1.5708 1.5708 1.5708" />
     </collision>
   </link>
@@ -106,7 +106,7 @@
     <collision>
       <geometry>
-        <mesh filename="package://clase5/robot_description/mycobot_320_m5_2022/link4.dae" />
-      </geometry>
-      <origin xyz="0.0 -0.0024 -0.05" rpy=" 1.5708 1.5708 0" />
+        <box size="0.0796 0.05932 0.0879" />
+      </geometry>
+      <origin xyz="-0.00002 -0.01367 -0.01055" rpy="1.5708 1.5708 0" />
     </collision>
   </link>
@@ -138,7 +138,7 @@
     <collision>
       <geometry>
-        <mesh filename="package://clase5/robot_description/mycobot_320_m5_2022/link6.dae" />
-      </geometry>
-      <origin xyz="0.0 0.0 -0.0115 " rpy=" 1.5708 1.5708 0" />
+        <box size="0.0192 0.05816 0.05816" />
+      </geometry>
+      <origin xyz="0.00010 -0.00020 -0.00165" rpy="1.5708 1.5708 0" />
     </collision>
   </link>
@@ -202,7 +202,7 @@
     <collision>
       <geometry>
-      <mesh filename="package://clase5/robot_description/adaptive_gripper/gripper_base.dae"/>
-      </geometry>
-    <origin xyz = "0.0 0 -0.012 " rpy = " 0 0 0"/>
+        <box size="0.058 0.07152 0.0537" />
+      </geometry>
+      <origin xyz="0 0.00644 -0.02005" rpy="0 0 0" />
     </collision>
   </link>
@@ -218,7 +218,7 @@
     <collision>
       <geometry>
-      <mesh filename="package://clase5/robot_description/adaptive_gripper/gripper_left1.dae"/>
-      </geometry>
-        <origin xyz = "0.039 -0.0133 -0.012 " rpy = " 0 0 0"/>
+        <box size="0.05926 0.02637 0.02233" />
+      </geometry>
+      <origin xyz="0.03687 -0.0133 -0.01117" rpy="0 0 0" />
     </collision>
   </link>
@@ -234,7 +234,7 @@
     <collision>
       <geometry>
-      <mesh filename="package://clase5/robot_description/adaptive_gripper/gripper_left2.dae"/>
-      </geometry>
-        <origin xyz = "0.005 -0.0195 -0.012 " rpy = " 0 0 0"/>
+        <box size="0.04001 0.02 0.009" />
+      </geometry>
+      <origin xyz="0.00497 -0.0226 -0.012" rpy="0 0 0" />
     </collision>
   </link>
@@ -250,7 +250,7 @@
     <collision>
       <geometry>
-      <mesh filename="package://clase5/robot_description/adaptive_gripper/gripper_left3.dae"/>
-      </geometry>
-    <origin xyz = "0.012 0.0025 -0.012 " rpy = " 0 0 0"/>
+        <box size="0.005 0.04017 0.04014" />
+      </geometry>
+      <origin xyz="0.0145 0.00834 -0.01785" rpy="0 0 0" />
     </collision>
   </link>
@@ -266,7 +266,7 @@
     <collision>
       <geometry>
-      <mesh filename="package://clase5/robot_description/adaptive_gripper/gripper_right1.dae"/>
-      </geometry>
-        <origin xyz = "-0.039 -0.0133 -0.012 " rpy = " 0 0 0"/>
+        <box size="0.05926 0.02637 0.02233" />
+      </geometry>
+      <origin xyz="-0.04113 -0.0133 -0.01117" rpy="0 0 0" />
     </collision>
   </link>
@@ -282,7 +282,7 @@
     <collision>
       <geometry>
-      <mesh filename="package://clase5/robot_description/adaptive_gripper/gripper_right2.dae"/>
-      </geometry>
-        <origin xyz = "-0.005 -0.0195 -0.012 " rpy = " 0 0 0"/>
+        <box size="0.04001 0.02 0.009" />
+      </geometry>
+      <origin xyz="-0.00503 -0.0226 -0.012" rpy="0 0 0" />
     </collision>
   </link>
@@ -298,7 +298,7 @@
     <collision>
       <geometry>
-      <mesh filename="package://clase5/robot_description/adaptive_gripper/gripper_right3.dae"/>
-      </geometry>
-    <origin xyz = "-0.012 0.0025 -0.012" rpy = " 0 0 0"/>
+        <box size="0.005 0.03576 0.0438" />
+      </geometry>
+      <origin xyz="-0.0095 0.00613 -0.01968" rpy="0 0 0" />
     </collision>
   </link>
@@ -376,5 +376,8 @@
        porque ros2_controllers.yaml ya define las ganancias PID por junta. -->
   <xacro:arg name="controllers_file" default="$(find clase5)/config/mycobot_320_m5_2022/ros2_controllers.yaml" />
-  <xacro:macro name="joint_control" params="joint">
+  <!-- Pose inicial: el brazo arranca plegado y estable, no estirado hacia
+       arriba, que es la pose desde la que se desploma. Coincide con el
+       group_state "listo" del SRDF. -->
+  <xacro:macro name="joint_control" params="joint init">
     <joint name="${joint}">
       <command_interface name="effort">
@@ -382,5 +385,7 @@
         <param name="max">${joint_effort}</param>
       </command_interface>
-      <state_interface name="position" />
+      <state_interface name="position">
+        <param name="initial_value">${init}</param>
+      </state_interface>
       <state_interface name="velocity" />
       <state_interface name="effort" />
@@ -391,10 +396,10 @@
       <plugin>gz_ros2_control/GazeboSimSystem</plugin>
     </hardware>
-    <xacro:joint_control joint="joint1" />
-    <xacro:joint_control joint="joint2" />
-    <xacro:joint_control joint="joint3" />
-    <xacro:joint_control joint="joint4" />
-    <xacro:joint_control joint="joint5" />
-    <xacro:joint_control joint="joint6" />
+    <xacro:joint_control joint="joint1" init="0.0" />
+    <xacro:joint_control joint="joint2" init="-0.6" />
+    <xacro:joint_control joint="joint3" init="1.2" />
+    <xacro:joint_control joint="joint4" init="0.0" />
+    <xacro:joint_control joint="joint5" init="-0.6" />
+    <xacro:joint_control joint="joint6" init="0.0" />
   </ros2_control>
   <gazebo>

Commit message: more minor changes

File: tp-final/clase5/robot_description/mycobot_320_m5_2022/mycobot_320_m5_2022.xacro (robot description, xacro)
@@ -14,4 +14,11 @@
   <xacro:property name="link6_mass" value="0.0739" />
   <xacro:property name="flange_mass" value="0.035" />
+  <!-- El motor de fisica (dartsim) no soporta constraints mimic: lo avisa con
+       "does not support mimic constraints, so no constraint will be created".
+       O sea que las cinco juntas mimic de la pinza quedan LIBRES. Sin friccion
+       se sacuden solas y ensucian la simulacion, asi que se las traba con
+       damping y friccion altos: la pinza no se acciona en este TP. -->
+  <xacro:property name="gripper_damping" value="5.0" />
+  <xacro:property name="gripper_friction" value="5.0" />
   <xacro:property name="gripper_base_mass" value="0.03" />
   <xacro:property name="gripper_finger_mass" value="0.008" />
@@ -314,4 +321,5 @@
     <child link="gripper_left3"/>
     <origin xyz= "-0.012 0.005 0" rpy = "0 0 0"/>
+    <dynamics damping="${gripper_damping}" friction="${gripper_friction}" />
   </joint>
   <joint name="gripper_base_to_gripper_left2" type="revolute">
@@ -322,4 +330,5 @@
     <origin xyz= "-0.005 0.027 0" rpy = "0 0 0"/>
     <mimic joint="gripper_controller" multiplier="1.0" offset="0" />
+    <dynamics damping="${gripper_damping}" friction="${gripper_friction}" />
   </joint>
   <joint name="gripper_left3_to_gripper_left1" type="revolute">
@@ -330,4 +339,5 @@
     <origin xyz= "-0.027 0.016 0" rpy = "0 0 0"/>
     <mimic joint="gripper_controller" multiplier="-1.0" offset="0" />
+    <dynamics damping="${gripper_damping}" friction="${gripper_friction}" />
   </joint>
   <joint name="gripper_base_to_gripper_right3" type="revolute">
@@ -338,4 +348,5 @@
     <origin xyz= "0.012 0.005 0" rpy = "0 0 0"/>
     <mimic joint="gripper_controller" multiplier="-1.0" offset="0" />
+    <dynamics damping="${gripper_damping}" friction="${gripper_friction}" />
   </joint>
   <joint name="gripper_base_to_gripper_right2" type="revolute">
@@ -346,4 +357,5 @@
     <origin xyz= "0.005 0.027 0" rpy = "0 0 0"/>
     <mimic joint="gripper_controller" multiplier="-1.0" offset="0" />
+    <dynamics damping="${gripper_damping}" friction="${gripper_friction}" />
   </joint>
   <joint name="gripper_right3_to_gripper_right1" type="revolute">
@@ -354,4 +366,5 @@
     <origin xyz= "0.027 0.016 0" rpy = "0 0 0"/>
     <mimic joint="gripper_controller" multiplier="1.0" offset="0" />
+    <dynamics damping="${gripper_damping}" friction="${gripper_friction}" />
   </joint>
   <!--  TCP / PUNTO DE AGARRE *******************-->
